File: PMOD_differential_driver.kicad_pcb (KiCad board)
At the start: 4 copper layers, 137.2 x 22.9 mm, 67 parts, among them J1 R/A 100mil Header 6x2, J2 RJ45_LED, J3 RJ45_LED, U1 SP3078EEN, U2 SP3078EEN, U3 SP3074EEN, U4 SP3074EEN

Commit message: Add files via upload
Parts:
- U3, U4: value SP3074EEN -> SP3078EEN
- moved TP16 2.18 mm to (125.9, 68.3)
Connections:
- JP3 pad 3: /SPI1_SCK_Z -> /SPI1_SCK_Y
- JP4 pad 3: /SPI1_SCK_Y -> /SPI1_SCK_Z
- JP5 pad 3: /SPI2_SCK_Z -> /SPI2_SCK_Y
- JP6 pad 3: /SPI2_SCK_Y -> /SPI2_SCK_Z
Routing:
- net /SPI2_SCK_Z: track 6.77 -> 15.1 mm, vias 0 -> 2
- net /SPI1_SCK_Z: track 8.42 -> 14.9 mm, vias 0 -> 2
- net /SPI2_SCK_Y: track 7.92 -> 11.5 mm
- net /SPI1_SCK_Y: track 11.4 -> 13.9 mm
- net /SPI2_SCK_1: track 124.4 -> 122.1 mm
- net GND: track 9.48 -> 10.3 mm, vias 87 -> 89
- net /SPI2_SCK_B: track 8.08 -> 7.42 mm, vias 2 -> 0
- net /SPI2_SCK: track 16.2 -> 15.6 mm
- net /SPI1_SDO: track 30.3 -> 29.8 mm
