File: PMOD_differential_driver.kicad_sch (KiCad schematic)
At the start: 67 parts, among them J1 R/A 100mil Header 6x2, J2 RJ45_LED, J3 RJ45_LED, U1 SP3078EEN, U2 SP3078EEN, U3 SP3074EEN, U4 SP3074EEN

Commit message: Add files via upload
Parts:
- U1, U2: value SP3078EEN -> SP3077EEN; LCSC C95362 -> C916162
- U3, U4: value SP3074EEN -> SP3077EEN; LCSC C30356 -> C916162
Connections:
- net SPI1_SCK_Y: now also JP3.3 (B); no longer JP4.3 (B)
- net SPI1_SCK_Z: now also JP4.3 (B); no longer JP3.3 (B)
- net SPI2_SCK_Y: now also JP5.3 (B); no longer JP6.3 (B)
- net SPI2_SCK_Z: now also JP6.3 (B); no longer JP5.3 (B)
Other:
- company: (none) -> UC Observatories
- title: (none) -> KASM Differential SPI Over Ethernet Board
Changed lines of the file:
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@@
 	(generator_version "8.0")
 	(paper "B")
+	(title_block
+		(title "KASM Differential SPI Over Ethernet Board")
+		(date "2024-07-16")
+		(rev "1")
+		(company "UC Observatories")
+	)
 	(junction
 		(at 288.29 201.93)
@@
 		)
 	)
+	(text "Client mode"
+		(exclude_from_sim no)
+		(at 217.678 110.998 0)
+		(effects
+			(font
+				(size 1.27 1.27)
+			)
+		)
+	)
 	(text "Host mode"
 		(exclude_from_sim no)
@@
 	(text "Client mode"
 		(exclude_from_sim no)
+		(at 217.678 85.344 0)
+		(effects
+			(font
+				(size 1.27 1.27)
+			)
+		)
+	)
+	(text "Client mode"
+		(exclude_from_sim no)
 		(at 217.932 225.552 0)
 		(effects
@@
 		)
 	)
+	(text "Host mode"
+		(exclude_from_sim no)
+		(at 217.17 95.504 0)
+		(effects
+			(font
+				(size 1.27 1.27)
+			)
+		)
+	)
 	(text "Jumper lets us choose whether\nwe are connecting to host \nside or client side.  \nHost side transmits clk, \nclient side receives clk"
 		(exclude_from_sim no)
@@
 	(text "Host mode"
 		(exclude_from_sim no)
+		(at 216.916 120.65 0)
+		(effects
+			(font
+				(size 1.27 1.27)
+			)
+		)
+	)
+	(text "Host mode"
+		(exclude_from_sim no)
 		(at 217.424 210.058 0)
 		(effects
@@
 		)
 	)
-	(label "SPI2_SCK_Z"
+	(label "SPI2_SCK_Y"
 		(at 212.09 208.28 0)
 		(fields_autoplaced yes)
@@
 		)
 	)
-	(label "SPI2_SCK_Y"
+	(label "SPI2_SCK_Z"
 		(at 212.09 233.68 0)
 		(fields_autoplaced yes)
@@
 		)
 	)
-	(label "SPI1_SCK_Z"
+	(label "SPI1_SCK_Y"
 		(at 212.09 93.98 0)
 		(fields_autoplaced yes)
@@
 		)
 	)
-	(label "SPI1_SCK_Y"
+	(label "SPI1_SCK_Z"
 		(at 212.09 119.38 0)
 		(fields_autoplaced yes)
@@
 			)
 		)
-		(property "Value" "SP3078EEN"
+		(property "Value" "SP3077EEN"
 			(at 140.6241 42.7298 0)
 			(effects
@@
 			)
 		)
-		(property "LCSC" "C95362"
+		(property "LCSC" "C916162"
 			(at 138.43 57.15 0)
 			(effects
@@
 			)
 		)
-		(property "Value" "SP3078EEN"
+		(property "Value" "SP3077EEN"
 			(at 140.6241 88.4498 0)
 			(effects
@@
 			)
 		)
-		(property "LCSC" "C95362"
+		(property "LCSC" "C916162"
 			(at 138.43 102.87 0)
 			(effects
@@
 			)
 		)
-		(property "Value" "SP3074EEN"
+		(property "Value" "SP3077EEN"
 			(at 140.6241 154.4898 0)
 			(effects
@@
 			)
 		)
-		(property "LCSC" "C30356"
+		(property "LCSC" "C916162"
 			(at 138.43 168.91 0)
 			(effects
@@
 			)
 		)
-		(property "Value" "SP3074EEN"
+		(property "Value" "SP3077EEN"
 			(at 140.6241 200.2098 0)
 			(effects
@@
 			)
 		)
-		(property "LCSC" "C30356"
+		(property "LCSC" "C916162"
 			(at 138.43 214.63 0)
 			(effects
